File: Open Source CDIs/DevSnapLock/DevSnapLock.kicad_sch (KiCad schematic)
At the start: 19 parts, among them J1 COIL, J2 MAG, J3 GtD, J4 AtG, J5 scrD, J6 lD, J7 aD, J8 aC, Q1 TIC106

Commit message: Added new CDIs and updated README
Added the DevPot_v2 CDI, updated the readme to include all of the new CDIs and included images for each. Also add production exports for all the boards.
Parts:
- C6: footprint Capacitor_THT:CP_Radial_Tantal_D5.5mm_P5.00mm -> Capacitor_THT:CP_Radial_Tantal_D5.5mm_P2.50mm
Changed lines of the file:
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@@
       (effects (font (size 1.27 1.27)) (justify right))
     )
-    (property "Footprint" "Capacitor_THT:CP_Radial_Tantal_D5.5mm_P5.00mm" (at 183.1848 102.87 0)
+    (property "Footprint" "Capacitor_THT:CP_Radial_Tantal_D5.5mm_P2.50mm" (at 183.1848 102.87 0)
       (effects (font (size 1.27 1.27)) hide)
     )
